File: pcb/openmv.brd (EAGLE design)
At the start: 35.6 x 26.7 mm, 5 parts

Commit message: eod
Parts:
- 24V: device con-molex:53047-02 -> pinhead:1X02
- moved 24V 1.28 mm to (3.81, 23.6)
Connections:
- removed net S$1: 24V.1, DC-DC5V.IN-.1, DC-DC5V.IN-.2
- net 3.3V: now also XPORT.2; no longer XPORT.7
- net GND: now also 24V.2, DC-DC5V.IN-.1, DC-DC5V.IN-.2, XPORT.1; no longer XPORT.8
- net S$2: now also 24V.1; no longer 24V.2
- net SCL: now also XPORT.5; no longer XPORT.4
- net SDA: now also XPORT.4; no longer XPORT.5
Routing:
- net S$1: track 10.6 -> 0.00 mm
- net S$2: track 25.0 -> 16.5 mm
- net SCL: track 18.6 -> 24.6 mm
- net SDA: track 22.2 -> 17.0 mm
- net GND: track 0.00 -> 2.54 mm
Other:
- board text added: "IOIA/ReverbLand2021"
- board text added: "rev0.2"
- board text removed: "IOIA/ReverbLand 2021"
Changed lines of the file:
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@@
 <text x="32.131" y="8.636" size="0.8128" layer="21" font="vector" ratio="22" rot="R90">P8</text>
 <text x="32.131" y="6.223" size="0.8128" layer="21" font="vector" ratio="22" rot="R90">P7</text>
-<text x="6.35" y="26.162" size="1.778" layer="16" rot="MR270">IOIA/ReverbLand 2021</text>
+<text x="30.48" y="18.796" size="1.016" layer="28" rot="MR270">IOIA/ReverbLand2021</text>
+<text x="8.763" y="0.762" size="1.016" layer="28" rot="MR0">rev0.2</text>
 </plain>
 <attributes>
@@
 <attribute name="VALUE" x="17.018" y="15.616" size="1.27" layer="28" rot="MR90"/>
 </element>
-<element name="24V" library="con-molex" library_urn="urn:adsk.eagle:library:165" package="53047-02" package3d_urn="urn:adsk.eagle:package:8078511/1" value="" x="2.54" y="23.495" smashed="yes" rot="MR0">
-<attribute name="NAME" x="4.415" y="25.245" size="1.27" layer="26" rot="MR0"/>
-<attribute name="VALUE" x="3.915" y="20.245" size="1.27" layer="28" rot="MR0"/>
-</element>
 <element name="IO" library="con-molex" library_urn="urn:adsk.eagle:library:165" package="53047-04" package3d_urn="urn:adsk.eagle:package:8078513/1" value="" x="32.131" y="23.495" smashed="yes" rot="MR0">
 <attribute name="NAME" x="35.256" y="25.245" size="1.27" layer="26" rot="MR0"/>
 <attribute name="VALUE" x="34.756" y="20.245" size="1.27" layer="28" rot="MR0"/>
+</element>
+<element name="24V" library="pinhead" library_urn="urn:adsk.eagle:library:325" package="1X02" package3d_urn="urn:adsk.eagle:package:22435/2" value="" x="3.81" y="23.622" smashed="yes" rot="MR0">
+<attribute name="NAME" x="6.4262" y="25.4508" size="1.27" layer="26" ratio="10" rot="MR0"/>
+<attribute name="VALUE" x="6.35" y="20.447" size="1.27" layer="28" rot="MR0"/>
 </element>
 </elements>
@@
 <contactref element="DC-DC5V" pad="OUT-.2"/>
 <contactref element="DC-DC5V" pad="OUT-.1"/>
-<contactref element="XPORT" pad="8"/>
 <contactref element="IO" pad="4"/>
+<contactref element="XPORT" pad="1"/>
+<contactref element="DC-DC5V" pad="IN-.1"/>
+<contactref element="DC-DC5V" pad="IN-.2"/>
+<wire x1="8.382" y1="21.717" x2="8.382" y2="19.177" width="0.3048" layer="1"/>
+<contactref element="24V" pad="2"/>
 </signal>
 <signal name="N$69">
@@
 <signal name="SDA">
 <contactref element="U$2" pad="16"/>
-<contactref element="XPORT" pad="5"/>
-<wire x1="1.651" y1="6.604" x2="2.54" y2="5.715" width="0.3048" layer="1"/>
-<wire x1="15.748" y1="5.715" x2="18.288" y2="8.255" width="0.3048" layer="1"/>
-<wire x1="18.288" y1="8.255" x2="18.288" y2="12.446" width="0.3048" layer="1"/>
-<wire x1="2.54" y1="5.715" x2="15.748" y2="5.715" width="0.3048" layer="1"/>
+<contactref element="XPORT" pad="4"/>
+<wire x1="1.651" y1="6.604" x2="3.54441875" y2="6.604" width="0.3048" layer="1"/>
+<wire x1="3.54441875" y1="6.604" x2="3.87461875" y2="6.2738" width="0.3048" layer="1"/>
+<wire x1="3.87461875" y1="6.2738" x2="13.3858" y2="6.2738" width="0.3048" layer="1"/>
+<wire x1="13.3858" y1="6.2738" x2="17.018" y2="9.906" width="0.3048" layer="1"/>
 </signal>
 <signal name="SCL">
 <contactref element="U$2" pad="15"/>
-<contactref element="XPORT" pad="4"/>
-<wire x1="1.651" y1="9.144" x2="4.191" y2="6.604" width="0.3048" layer="1"/>
-<wire x1="4.191" y1="6.604" x2="15.113" y2="6.604" width="0.3048" layer="1"/>
-<wire x1="15.113" y1="6.604" x2="17.018" y2="8.509" width="0.3048" layer="1"/>
-<wire x1="17.018" y1="8.509" x2="17.018" y2="9.906" width="0.3048" layer="1"/>
+<contactref element="XPORT" pad="5"/>
+<wire x1="1.651" y1="9.144" x2="4.064" y2="6.731" width="0.3048" layer="1"/>
+<wire x1="4.064" y1="6.731" x2="10.541" y2="6.731" width="0.3048" layer="1"/>
+<wire x1="10.541" y1="6.731" x2="11.43" y2="7.62" width="0.3048" layer="1"/>
+<wire x1="11.43" y1="7.62" x2="11.43" y2="13.716" width="0.3048" layer="1"/>
+<wire x1="11.43" y1="13.716" x2="17.018" y2="13.716" width="0.3048" layer="1"/>
+<wire x1="17.018" y1="13.716" x2="18.288" y2="12.446" width="0.3048" layer="1"/>
 </signal>
 <signal name="3.3V">
 <contactref element="U$2" pad="18"/>
-<contactref element="XPORT" pad="7"/>
-<wire x1="1.651" y1="1.524" x2="10.48255625" y2="1.524" width="0.3048" layer="1"/>
-<wire x1="10.48255625" y1="1.524" x2="10.60895625" y2="1.3976" width="0.3048" layer="1"/>
-<wire x1="10.60895625" y1="1.3976" x2="14.3516" y2="1.3976" width="0.3048" layer="1"/>
-<wire x1="14.3516" y1="1.3976" x2="20.828" y2="7.874" width="0.3048" layer="1"/>
-<wire x1="20.828" y1="7.874" x2="20.828" y2="12.446" width="0.3048" layer="1"/>
+<contactref element="XPORT" pad="2"/>
+<wire x1="18.415" y1="10.668" x2="17.78" y2="11.303" width="0.3048" layer="1"/>
+<wire x1="17.78" y1="11.303" x2="15.875" y2="11.303" width="0.3048" layer="1"/>
+<wire x1="15.875" y1="11.303" x2="14.478" y2="9.906" width="0.3048" layer="1"/>
+<wire x1="1.651" y1="1.524" x2="5.9436" y2="5.8166" width="0.3048" layer="1"/>
+<wire x1="5.9436" y1="5.8166" x2="13.57518125" y2="5.8166" width="0.3048" layer="1"/>
+<wire x1="16.26758125" y1="8.509" x2="18.034" y2="8.509" width="0.3048" layer="1"/>
+<wire x1="13.57518125" y1="5.8166" x2="16.26758125" y2="8.509" width="0.3048" layer="1"/>
+<wire x1="18.034" y1="8.509" x2="18.415" y2="8.89" width="0.3048" layer="1"/>
+<wire x1="18.415" y1="8.89" x2="18.415" y2="10.668" width="0.3048" layer="1"/>
 </signal>
 <signal name="N$1">
@@
 <contactref element="U$2" pad="23"/>
 </signal>
-<signal name="S$1">
-<contactref element="DC-DC5V" pad="IN-.1"/>
-<contactref element="DC-DC5V" pad="IN-.2"/>
-<contactref element="24V" pad="1"/>
-<wire x1="8.382" y1="21.717" x2="8.382" y2="19.177" width="0.3048" layer="1"/>
-<wire x1="1.915" y1="23.945" x2="1.915" y2="22.723" width="0.3048" layer="1"/>
-<wire x1="2.921" y1="21.717" x2="8.382" y2="21.717" width="0.3048" layer="1"/>
-<wire x1="1.915" y1="22.723" x2="2.921" y2="21.717" width="0.3048" layer="1"/>
-</signal>
 <signal name="S$2">
 <contactref element="DC-DC5V" pad="IN+.1"/>
 <contactref element="DC-DC5V" pad="IN+.2"/>
-<contactref element="24V" pad="2"/>
 <wire x1="8.382" y1="8.509" x2="8.382" y2="11.049" width="0.3048" layer="1"/>
-<wire x1="8.382" y1="11.049" x2="8.001" y2="11.43" width="0.3048" layer="1"/>
-<wire x1="8.001" y1="11.43" x2="8.001" y2="17.272" width="0.3048" layer="1"/>
-<wire x1="8.001" y1="17.272" x2="8.128" y2="17.399" width="0.3048" layer="1"/>
-<wire x1="8.128" y1="17.399" x2="10.414" y2="17.399" width="0.3048" layer="1"/>
-<wire x1="10.414" y1="17.399" x2="10.414" y2="23.622" width="0.3048" layer="1"/>
-<wire x1="10.414" y1="23.622" x2="10.091" y2="23.945" width="0.3048" layer="1"/>
-<wire x1="10.091" y1="23.945" x2="3.165" y2="23.945" width="0.3048" layer="1"/>
+<contactref element="24V" pad="1"/>
+<wire x1="5.08" y1="23.622" x2="5.08" y2="14.351" width="0.3048" layer="1"/>
+<wire x1="5.08" y1="14.351" x2="8.382" y2="11.049" width="0.3048" layer="1"/>
 </signal>
 </signals>
@@
 <mfgpreviewcolor name="substratecolor" color="0xFF786E46"/>
 </mfgpreviewcolors>
-<errors>
-</errors>
 </board>
 </drawing>

Commit message: eod
Parts:
- removed 24V: (no value), pinhead:1X02
- removed IO: (no value), con-molex:53047-04
- added E$1, E$2: (no value), con-lstb:MA04-1
Connections:
- net GND: now also E$1.2, E$2.2; no longer 24V.2, IO.4
- net MISO: now also E$1.4
- net MOSI: now also E$1.3; no longer IO.1
- net PWM1: now also E$2.3; no longer IO.2
- net PWM2: now also E$2.4; no longer IO.3
- net S$2: now also E$1.1, E$2.1; no longer 24V.1
Routing:
- net MOSI: track 37.2 -> 8.63 mm
- net GND: track 2.54 -> 29.4 mm
- net S$2: track 16.5 -> 42.5 mm
- net MISO: track 0.00 -> 16.4 mm
- net PWM2: track 15.6 -> 18.4 mm
- net PWM1: track 18.3 -> 20.3 mm
- net SDA: track 17.0 -> 18.4 mm
Other:
- board size 35.6 x 26.7 mm -> 35.6 x 27.7 mm
Changed lines of the file:
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@@
 <plain>
 <wire x1="0" y1="0" x2="35.56" y2="0" width="0" layer="20"/>
-<wire x1="35.56" y1="0" x2="35.56" y2="26.67" width="0" layer="20"/>
-<wire x1="35.56" y1="26.67" x2="0" y2="26.67" width="0" layer="20"/>
-<wire x1="0" y1="26.67" x2="0" y2="0" width="0" layer="20"/>
+<wire x1="35.56" y1="0" x2="35.56" y2="27.686" width="0" layer="20"/>
+<wire x1="35.56" y1="27.686" x2="0" y2="27.686" width="0" layer="20"/>
+<wire x1="0" y1="27.686" x2="0" y2="0" width="0" layer="20"/>
 <text x="3.429" y="3.302" size="0.8128" layer="22" font="vector" ratio="22" rot="MR90">P6</text>
 <text x="3.429" y="8.382" size="0.8128" layer="22" font="vector" ratio="22" rot="MR90">P4</text>
@@
 <attribute name="VALUE" x="17.018" y="15.616" size="1.27" layer="28" rot="MR90"/>
 </element>
-<element name="IO" library="con-molex" library_urn="urn:adsk.eagle:library:165" package="53047-04" package3d_urn="urn:adsk.eagle:package:8078513/1" value="" x="32.131" y="23.495" smashed="yes" rot="MR0">
-<attribute name="NAME" x="35.256" y="25.245" size="1.27" layer="26" rot="MR0"/>
-<attribute name="VALUE" x="34.756" y="20.245" size="1.27" layer="28" rot="MR0"/>
+<element name="E$1" library="con-lstb" library_urn="urn:adsk.eagle:library:162" package="MA04-1" package3d_urn="urn:adsk.eagle:package:8337/1" value="" x="5.588" y="25.781" smashed="yes">
+<attribute name="NAME" x="0.508" y="27.432" size="1.27" layer="25" ratio="10"/>
+<attribute name="VALUE" x="6.223" y="27.432" size="1.27" layer="27" ratio="10"/>
 </element>
-<element name="24V" library="pinhead" library_urn="urn:adsk.eagle:library:325" package="1X02" package3d_urn="urn:adsk.eagle:package:22435/2" value="" x="3.81" y="23.622" smashed="yes" rot="MR0">
-<attribute name="NAME" x="6.4262" y="25.4508" size="1.27" layer="26" ratio="10" rot="MR0"/>
-<attribute name="VALUE" x="6.35" y="20.447" size="1.27" layer="28" rot="MR0"/>
+<element name="E$2" library="con-lstb" library_urn="urn:adsk.eagle:library:162" package="MA04-1" package3d_urn="urn:adsk.eagle:package:8337/1" value="" x="29.972" y="25.781" smashed="yes">
+<attribute name="NAME" x="24.892" y="27.432" size="1.27" layer="25" ratio="10"/>
+<attribute name="VALUE" x="30.607" y="27.432" size="1.27" layer="27" ratio="10"/>
 </element>
 </elements>
@@
 <vertex x="0" y="0"/>
 <vertex x="35.56" y="0"/>
-<vertex x="35.56" y="26.67"/>
-<vertex x="0" y="26.67"/>
+<vertex x="35.56" y="27.686"/>
+<vertex x="0" y="27.686"/>
 </polygon>
 <polygon width="0.3048" layer="1" isolate="0.3048" rank="2">
 <vertex x="0" y="0"/>
 <vertex x="35.56" y="0"/>
-<vertex x="35.56" y="26.67"/>
-<vertex x="0" y="26.67"/>
+<vertex x="35.56" y="27.686"/>
+<vertex x="0" y="27.686"/>
 </polygon>
 <contactref element="DC-DC5V" pad="OUT-.2"/>
 <contactref element="DC-DC5V" pad="OUT-.1"/>
-<contactref element="IO" pad="4"/>
 <contactref element="XPORT" pad="1"/>
 <contactref element="DC-DC5V" pad="IN-.1"/>
 <contactref element="DC-DC5V" pad="IN-.2"/>
 <wire x1="8.382" y1="21.717" x2="8.382" y2="19.177" width="0.3048" layer="1"/>
-<contactref element="24V" pad="2"/>
+<contactref element="E$1" pad="2"/>
+<contactref element="E$2" pad="2"/>
+<wire x1="33.909" y1="1.524" x2="28.829" y2="6.604" width="0.3048" layer="1"/>
+<wire x1="28.829" y1="6.604" x2="25.654" y2="6.604" width="0.3048" layer="1"/>
+<wire x1="25.654" y1="6.604" x2="25.273" y2="6.985" width="0.3048" layer="1"/>
+<wire x1="26.2702" y1="13.9512" x2="26.3013125" y2="13.9512" width="0.3048" layer="1"/>
+<wire x1="26.3013125" y1="13.9512" x2="27.559" y2="15.2088875" width="0.3048" layer="1"/>
+<wire x1="27.559" y1="18.542" x2="26.924" y2="19.177" width="0.3048" layer="1"/>
+<wire x1="25.273" y1="6.985" x2="25.273" y2="12.954" width="0.3048" layer="1"/>
+<wire x1="25.273" y1="12.954" x2="26.2702" y2="13.9512" width="0.3048" layer="1"/>
+<wire x1="27.559" y1="15.2088875" x2="27.559" y2="18.542" width="0.3048" layer="1"/>
+<wire x1="26.924" y1="19.177" x2="26.924" y2="21.717" width="0.3048" layer="1"/>
+<wire x1="13.208" y1="12.446" x2="8.382" y2="19.177" width="0" layer="19" extent="1-1"/>
 </signal>
 <signal name="N$69">
@@
 <wire x1="1.651" y1="6.604" x2="3.54441875" y2="6.604" width="0.3048" layer="1"/>
 <wire x1="3.54441875" y1="6.604" x2="3.87461875" y2="6.2738" width="0.3048" layer="1"/>
-<wire x1="3.87461875" y1="6.2738" x2="13.3858" y2="6.2738" width="0.3048" layer="1"/>
-<wire x1="13.3858" y1="6.2738" x2="17.018" y2="9.906" width="0.3048" layer="1"/>
+<wire x1="15.5702" y1="6.2738" x2="15.621" y2="6.223" width="0.3048" layer="1"/>
+<wire x1="3.87461875" y1="6.2738" x2="15.5702" y2="6.2738" width="0.3048" layer="1"/>
+<wire x1="15.621" y1="6.223" x2="17.018" y2="7.62" width="0.3048" layer="1"/>
+<wire x1="17.018" y1="7.62" x2="17.018" y2="9.906" width="0.3048" layer="1"/>
 </signal>
 <signal name="SCL">
@@
 <contactref element="U$2" pad="18"/>
 <contactref element="XPORT" pad="2"/>
-<wire x1="18.415" y1="10.668" x2="17.78" y2="11.303" width="0.3048" layer="1"/>
-<wire x1="17.78" y1="11.303" x2="15.875" y2="11.303" width="0.3048" layer="1"/>
-<wire x1="15.875" y1="11.303" x2="14.478" y2="9.906" width="0.3048" layer="1"/>
-<wire x1="1.651" y1="1.524" x2="5.9436" y2="5.8166" width="0.3048" layer="1"/>
-<wire x1="5.9436" y1="5.8166" x2="13.57518125" y2="5.8166" width="0.3048" layer="1"/>
-<wire x1="16.26758125" y1="8.509" x2="18.034" y2="8.509" width="0.3048" layer="1"/>
-<wire x1="13.57518125" y1="5.8166" x2="16.26758125" y2="8.509" width="0.3048" layer="1"/>
-<wire x1="18.034" y1="8.509" x2="18.415" y2="8.89" width="0.3048" layer="1"/>
-<wire x1="18.415" y1="8.89" x2="18.415" y2="10.668" width="0.3048" layer="1"/>
+<wire x1="18.415" y1="10.033" x2="17.272" y2="11.176" width="0.3048" layer="1"/>
+<wire x1="17.272" y1="11.176" x2="15.748" y2="11.176" width="0.3048" layer="1"/>
+<wire x1="15.748" y1="11.176" x2="14.478" y2="9.906" width="0.3048" layer="1"/>
+<wire x1="1.651" y1="1.524" x2="5.842" y2="5.715" width="0.3048" layer="1"/>
+<wire x1="5.842" y1="5.715" x2="16.764" y2="5.715" width="0.3048" layer="1"/>
+<wire x1="16.764" y1="5.715" x2="18.415" y2="7.366" width="0.3048" layer="1"/>
+<wire x1="18.415" y1="7.366" x2="18.415" y2="10.033" width="0.3048" layer="1"/>
 </signal>
 <signal name="N$1">
@@
 <signal name="MOSI">
 <contactref element="U$2" pad="11"/>
-<contactref element="IO" pad="1"/>
-<wire x1="1.651" y1="19.304" x2="0.762" y2="20.193" width="0.3048" layer="1"/>
-<wire x1="0.762" y1="20.193" x2="0.762" y2="25.273" width="0.3048" layer="1"/>
-<wire x1="0.762" y1="25.273" x2="1.27" y2="25.781" width="0.3048" layer="1"/>
-<wire x1="1.27" y1="25.781" x2="29.083" y2="25.781" width="0.3048" layer="1"/>
-<wire x1="29.083" y1="25.781" x2="30.256" y2="24.608" width="0.3048" layer="1"/>
-<wire x1="30.256" y1="24.608" x2="30.256" y2="23.945" width="0.3048" layer="1"/>
+<contactref element="E$1" pad="3"/>
+<wire x1="1.651" y1="19.304" x2="6.858" y2="24.511" width="0.3048" layer="1"/>
+<wire x1="6.858" y1="24.511" x2="6.858" y2="25.781" width="0.3048" layer="1"/>
 </signal>
 <signal name="PWM2">
 <contactref element="U$2" pad="25"/>
-<contactref element="IO" pad="3"/>
-<wire x1="33.909" y1="9.144" x2="32.385" y2="10.668" width="0.3048" layer="1"/>
-<wire x1="32.756" y1="22.342" x2="32.756" y2="23.945" width="0.3048" layer="1"/>
-<wire x1="32.385" y1="10.668" x2="32.385" y2="21.971" width="0.3048" layer="1"/>
-<wire x1="32.385" y1="21.971" x2="32.756" y2="22.342" width="0.3048" layer="1"/>
+<contactref element="E$2" pad="4"/>
+<wire x1="33.909" y1="9.144" x2="31.6992" y2="11.3538" width="0.3048" layer="1"/>
+<wire x1="31.6992" y1="23.6982" x2="33.782" y2="25.781" width="0.3048" layer="1"/>
+<wire x1="31.6992" y1="11.3538" x2="31.6992" y2="23.6982" width="0.3048" layer="1"/>
 </signal>
 <signal name="PWM1">
 <contactref element="U$2" pad="26"/>
-<contactref element="IO" pad="2"/>
-<wire x1="33.909" y1="6.604" x2="31.506" y2="9.007" width="0.3048" layer="1"/>
-<wire x1="31.506" y1="9.007" x2="31.506" y2="23.945" width="0.3048" layer="1"/>
+<contactref element="E$2" pad="3"/>
+<wire x1="33.909" y1="6.604" x2="31.242" y2="9.271" width="0.3048" layer="1"/>
+<wire x1="31.242" y1="9.271" x2="31.242" y2="25.781" width="0.3048" layer="1"/>
 </signal>
 <signal name="VIN">
@@
 <signal name="MISO">
 <contactref element="U$2" pad="12"/>
+<contactref element="E$1" pad="4"/>
+<wire x1="1.651" y1="16.764" x2="8.255" y2="16.764" width="0.3048" layer="1"/>
+<wire x1="8.255" y1="16.764" x2="9.779" y2="18.288" width="0.3048" layer="1"/>
+<wire x1="9.779" y1="18.288" x2="9.779" y2="25.4" width="0.3048" layer="1"/>
+<wire x1="9.779" y1="25.4" x2="9.398" y2="25.781" width="0.3048" layer="1"/>
 </signal>
 <signal name="SWC">
@@
 <contactref element="DC-DC5V" pad="IN+.2"/>
 <wire x1="8.382" y1="8.509" x2="8.382" y2="11.049" width="0.3048" layer="1"/>
-<contactref element="24V" pad="1"/>
-<wire x1="5.08" y1="23.622" x2="5.08" y2="14.351" width="0.3048" layer="1"/>
-<wire x1="5.08" y1="14.351" x2="8.382" y2="11.049" width="0.3048" layer="1"/>
+<contactref element="E$1" pad="1"/>
+<contactref element="E$2" pad="1"/>
+<wire x1="8.382" y1="11.049" x2="5.334" y2="14.097" width="0.4064" layer="16"/>
+<wire x1="5.334" y1="20.828" x2="1.778" y2="24.384" width="0.4064" layer="16"/>
+<wire x1="5.334" y1="14.097" x2="5.334" y2="20.828" width="0.4064" layer="16"/>
+<wire x1="8.382" y1="11.049" x2="23.114" y2="25.781" width="0.4064" layer="16"/>
+<wire x1="23.114" y1="25.781" x2="26.162" y2="25.781" width="0.4064" layer="16"/>
+<wire x1="1.778" y1="24.384" x2="1.778" y2="25.781" width="0" layer="19" extent="16-16"/>
 </signal>
 </signals>
